File: pcb_files/xt_pcb/xt_pcb.kicad_pcb (KiCad board)
At the start: 2 copper layers, 400.1 x 95.2 mm, 211 parts, among them J1 Conn_01x04_Socket, J2 Conn_01x05, J3 USB_C_Receptacle_USB2.0, SW1 SW_Push, SW10 SW_Push, SW11 SW_Push, SW12 SW_Push, SW13 SW_Push, SW14 SW_Push, SW15 SW_Push, SW16 SW_Push, SW17 SW_Push, SW18 SW_Push, SW19 SW_Push, SW20 SW_Push, SW21 SW_Push, SW22 SW_Push, SW23 SW_Push, SW24 SW_Push, SW25 SW_Push, SW26 SW_Push, SW27 SW_Push, SW28 SW_Push, SW29 SW_Push, SW3 SW_Push, SW30 SW_Push, SW31 SW_Push, SW32 SW_Push, SW33 SW_Push, SW34 SW_Push, SW35 SW_Push, SW36 SW_Push, SW37 SW_Push, SW38 SW_Push, SW39 SW_Push, SW4 SW_Push, SW40 SW_Push, SW41 SW_Push, SW42 SW_Push, SW43 SW_Push, SW44 SW_Push, SW45 SW_Push, SW46 SW_Push, SW47 SW_Push, SW48 SW_Push, SW49 SW_Push, SW5 SW_Push, SW50 SW_Push, SW51 SW_Push, SW52 SW_Push, SW53 SW_Push, SW54 SW_Push, SW55 SW_Push, SW56 SW_Push, SW57 SW_Push, SW58 SW_Push, SW59 SW_Push, SW6 SW_Push, SW60 SW_Push, SW61 SW_Push, SW62 SW_Push, SW64 SW_Push, SW66 SW_Push, SW67 SW_Push, SW68 SW_Push, SW69 SW_Push, SW7 SW_Push, SW70 SW_Push, SW71 SW_Push, SW72 SW_Push, SW73 SW_Push, SW74 SW_Push, SW75 SW_Push, SW76 SW_Push, SW77 SW_Push, SW78 SW_Push, SW79 SW_Push, SW8 SW_Push, SW80 SW_Push, SW81 SW_Push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

Commit message: debugging + prod files
Routing:
- net GND: track 150.0 -> 151.9 mm, vias 26 -> 27
Changed lines of the file:
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@@
+	)
+	(segment
+		(start 112.4815 89.575)
+		(end 112.4815 91.945)
+		(width 0.2)
+		(layer "F.Cu")
+		(net 2)
 	)
 	(segment
@@
 	)
 	(segment
-		(start 112.4815 89.575)
+		(start 112.4815 91.945)
 		(end 112.4815 92.445)
 		(width 0.2)
@@
 	)
 	(via
+		(at 112.4815 91.945)
+		(size 0.6)
+		(drill 0.3)
+		(layers "F.Cu" "B.Cu")
+		(net 2)
+	)
+	(via
 		(at 230.3315 162.505)
 		(size 0.6)
@@
 		(width 0.2)
 		(layer "B.Cu")
+		(net 2)
+	)
+	(segment
+		(start 111.4115 90.49)
+		(end 111.4115 90.875)
+		(width 0.2)
+		(layer "B.Cu")
+		(net 2)
+	)
+	(segment
+		(start 111.4115 90.875)
+		(end 112.4815 91.945)
+		(width 0.2)
+		(layer "B.Cu")

Commit message: rerouting
Routing:
- net GND: track 151.9 -> 121.0 mm, vias 27 -> 29
- net R3: track 541.7 -> 524.0 mm, vias 10 -> 7
- net C16: track 266.8 -> 250.1 mm
- net C12: track 186.2 -> 176.6 mm, vias 1 -> 0
- net R1: track 550.0 -> 540.6 mm
- net C7: track 109.4 -> 114.5 mm, vias 1 -> 0
- net C9: track 111.4 -> 106.3 mm
- net C13: track 217.4 -> 214.0 mm
- net C8: track 138.7 -> 135.6 mm
- net C5: track 142.5 -> 140.0 mm
- net C1: track 234.8 -> 233.1 mm
- net C4: track 167.2 -> 165.6 mm
- net C3: track 201.6 -> 200.1 mm
- net C19: track 322.5 -> 323.9 mm
- net C17: track 276.3 -> 274.9 mm
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
Commit message: removed all 90 deg
Routing:
- net R3: track 524.0 -> 506.1 mm
- net C12: track 176.6 -> 183.8 mm, vias 0 -> 1
- net C2: track 222.0 -> 216.3 mm
- net C18: track 304.8 -> 302.0 mm
- net C19: track 323.9 -> 321.1 mm
- net Net-(D68-A): track 30.2 -> 29.0 mm
- net Q_IO2: track 21.9 -> 21.1 mm
- net C7: track 114.5 -> 113.8 mm
- net C11: track 130.5 -> 129.9 mm
