File: pcb_files/xt_pcb/_autosave-xt_pcb.kicad_pcb (KiCad board)
At the start: 2 copper layers, 400.1 x 95.2 mm, 211 parts, among them J1 Conn_01x04_Socket, J2 Conn_01x05, J3 USB_C_Receptacle_USB2.0, SW1 SW_Push, SW10 SW_Push, SW11 SW_Push, SW12 SW_Push, SW13 SW_Push, SW14 SW_Push, SW15 SW_Push, SW16 SW_Push, SW17 SW_Push, SW18 SW_Push, SW19 SW_Push, SW20 SW_Push, SW21 SW_Push, SW22 SW_Push, SW23 SW_Push, SW24 SW_Push, SW25 SW_Push, SW26 SW_Push, SW27 SW_Push, SW28 SW_Push, SW29 SW_Push, SW3 SW_Push, SW30 SW_Push, SW31 SW_Push, SW32 SW_Push, SW33 SW_Push, SW34 SW_Push, SW35 SW_Push, SW36 SW_Push, SW37 SW_Push, SW38 SW_Push, SW39 SW_Push, SW4 SW_Push, SW40 SW_Push, SW41 SW_Push, SW42 SW_Push, SW43 SW_Push, SW44 SW_Push, SW45 SW_Push, SW46 SW_Push, SW47 SW_Push, SW48 SW_Push, SW49 SW_Push, SW5 SW_Push, SW50 SW_Push, SW51 SW_Push, SW52 SW_Push, SW53 SW_Push, SW54 SW_Push, SW55 SW_Push, SW56 SW_Push, SW57 SW_Push, SW58 SW_Push, SW59 SW_Push, SW6 SW_Push, SW60 SW_Push, SW61 SW_Push, SW62 SW_Push, SW64 SW_Push, SW66 SW_Push, SW67 SW_Push, SW68 SW_Push, SW69 SW_Push, SW7 SW_Push, SW70 SW_Push, SW71 SW_Push, SW72 SW_Push, SW73 SW_Push, SW74 SW_Push, SW75 SW_Push, SW76 SW_Push, SW77 SW_Push, SW78 SW_Push, SW79 SW_Push, SW8 SW_Push, SW80 SW_Push, SW81 SW_Push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

Commit message: keyboard.json
Parts:
- SW96: footprint PCM_Switch_Keyboard_Hotswap_Kailh:SW_Hotswap_Kailh_MX_Plated_2.75u -> PCM_Switch_Keyboard_Hotswap_Kailh:SW_Hotswap_Kailh_MX_Plated_1.75u
Changed lines of the file:
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@@
 		)
 	)
-	(footprint "PCM_Switch_Keyboard_Hotswap_Kailh:SW_Hotswap_Kailh_MX_Plated_2.75u"
+	(footprint "PCM_Switch_Keyboard_Hotswap_Kailh:SW_Hotswap_Kailh_MX_Plated_1.75u"
 		(layer "F.Cu")
 		(at 363.60625 147.605)
-		(descr "Kailh keyswitch Hotswap Socket plated holes Keycap 2.75u")
-		(tags "Kailh Keyboard Keyswitch Switch Hotswap Socket Plated Relief Cutout Keycap 2.75u")
+		(descr "Kailh keyswitch Hotswap Socket plated holes Keycap 1.75u")
+		(tags "Kailh Keyboard Keyswitch Switch Hotswap Socket Plated Relief Cutout Keycap 1.75u")
 		(property "Reference" "SW96"
 			(at 0 -8 0)
@@
 			)
 		)
-		(property "Datasheet" "~"
+		(property "Datasheet" ""
 			(at 0 0 0)
 			(layer "F.Fab")
@@
 			)
 		)
-		(property "Description" "Push button switch, generic, two pins"
+		(property "Description" ""
 			(at 0 0 0)
 			(layer "F.Fab")
@@
 		)
 		(fp_line
-			(start -26.19375 -9.525)
-			(end -26.19375 9.525)
+			(start -16.66875 -9.525)
+			(end -16.66875 9.525)
 			(stroke
 				(width 0.1)
@@
 		)
 		(fp_line
-			(start -26.19375 9.525)
-			(end 26.19375 9.525)
+			(start -16.66875 9.525)
+			(end 16.66875 9.525)
 			(stroke
 				(width 0.1)
@@
 		)
 		(fp_line
-			(start 26.19375 -9.525)
-			(end -26.19375 -9.525)
+			(start 16.66875 -9.525)
+			(end -16.66875 -9.525)
 			(stroke
 				(width 0.1)
@@
 		)
 		(fp_line
-			(start 26.19375 9.525)
-			(end 26.19375 -9.525)
+			(start 16.66875 9.525)
+			(end 16.66875 -9.525)
 			(stroke
 				(width 0.1)
